File: hw/main_board.sch (EAGLE design)
At the start: 86 parts, among them IC1 MCP3202SN, Q1 IRFR5305, Q2 IRFR5305, Q3 2N7002, Q4 Si4134, SW1 EC12E_SW, T1 BC807, T2 BC817, T3 BC817, U2 ESP-WROOM-32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

Commit message: Shrinked schematic to A4 paper
Other:
- note added: "17.10.2018"
- note added: "Martin Kousal"
